File: LED-strip_90.0x3.6mm__panel-v-cut.kicad_pcb (KiCad board)
At the start: 2 copper layers, 99 x 100 mm, 474 parts, among them P1 CONN_2, P2 CONN_2, P3 CONN_2, P4 CONN_2, P5 CONN_2, P6 CONN_2

Commit message: Added commit-ID to gerber files of the panel (fdf2c798...).
Other:
- board text added: "LED-strip_90.0x3.6mm"
- board text added: "commit fdf2c798cf86a2aec945da4a4678425f73c75afd"
