File: LED-strip_90x4mm.kicad_pcb (KiCad board)
At the start: 2 copper layers, 4 x 90 mm, 20 parts, among them P1 CONN_2, P2 CONN_2, P3 CONN_2, P4 CONN_2, P5 CONN_2, P6 CONN_2

Commit message: Duplicated F_Cu to B_Cu.
Parts:
- added D10: LED, my_parts:MADW__CHIPLED-0805, B.Cu at (200.0, 60.0)
- added D11: LED, my_parts:MADW__CHIPLED-0805, B.Cu at (200.0, 70.0)
- added D12: LED, my_parts:MADW__CHIPLED-0805, B.Cu at (200.0, 80.0)
- added D13: LED, my_parts:MADW__CHIPLED-0805, B.Cu at (200.0, 90.0)
- added D14: LED, my_parts:MADW__CHIPLED-0805, B.Cu at (200.0, 100.0)
- added D15: LED, my_parts:MADW__CHIPLED-0805, B.Cu at (200.0, 110.0)
- added D16: LED, my_parts:MADW__CHIPLED-0805, B.Cu at (200.0, 120.0)
- added D17: LED, my_parts:MADW__CHIPLED-0805, B.Cu at (200.0, 130.0)
- added D18: LED, my_parts:MADW__CHIPLED-0805, B.Cu at (200.0, 140.0)
- added P10: CONN_2, my_parts:MADW__SIL-2, B.Cu at (200.0, 113.5)
- added P11: CONN_2, my_parts:MADW__SIL-2, B.Cu at (200.0, 116.5)
- added P12: CONN_2, my_parts:MADW__SIL-2, B.Cu at (200.0, 143.5)
- added P7: CONN_2, my_parts:MADW__SIL-2, B.Cu at (200.0, 56.5)
- added P8: CONN_2, my_parts:MADW__SIL-2, B.Cu at (200.0, 83.5)
- added P9: CONN_2, my_parts:MADW__SIL-2, B.Cu at (200.0, 86.5)
- added R4: R, my_parts:MADW__R0603_2, B.Cu at (200.0, 74.9)
- added R5: R, my_parts:MADW__R0603_2, B.Cu at (200.0, 104.9)
- added R6: R, my_parts:MADW__R0603_2, B.Cu at (200.0, 134.9)
- moved G1 8.10 mm to (200.1, 65.1)
- moved G2 5.05 mm to (200.0, 95.0)
Routing:
- net /GND: track 94.7 -> 200.3 mm, vias 0 -> 1
- net /VCC: track 96.0 -> 198.3 mm, vias 0 -> 1
- net Net-(D13-Pad2): track 0.00 -> 7.90 mm
- net Net-(D10-Pad2): track 0.00 -> 7.90 mm
- net Net-(D16-Pad2): track 0.00 -> 7.90 mm
- net Net-(D18-Pad1): track 0.00 -> 3.20 mm
- net Net-(D15-Pad1): track 0.00 -> 3.20 mm
- net Net-(D12-Pad1): track 0.00 -> 3.20 mm
- net Net-(D14-Pad2): track 0.00 -> 3.00 mm
- net Net-(D11-Pad2): track 0.00 -> 3.00 mm
- net Net-(D17-Pad2): track 0.00 -> 3.00 mm
Other:
- net class Default: clearance 0.1524 -> 0.2032
- net class Power: clearance 0.1524 -> 0.2032
- rule trace_clearance: 0.1524 -> 0.2032
- rule via_min_drill: 0.3 -> 0.3302
- rule via_min_size: 0.6 -> 0.635
- board text added: "2014 V0.20.a"
- board text removed: "+ -"
- board text removed: "2014 - blog.spitzenpfeil.org"
- board text removed: "V0.10.b"
