File: LED-strip_90x4mm__panel-v-cut.kicad_pcb (KiCad board)
At the start: 2 copper layers, 99 x 100 mm, 414 parts, among them P1 CONN_2, P2 CONN_2, P3 CONN_2, P4 CONN_2, P5 CONN_2, P6 CONN_2

Commit message: Tweaks.
Parts:
- removed the G1 at (304.5, 90.0)
- removed the G1 at (324.5, 90.0)
- removed the G1 at (364.5, 90.0)
- removed the G1 at (368.5, 90.0)
- removed the G1 at (360.5, 90.0)
- removed the G1 at (356.5, 90.0)
- removed the G1 at (352.5, 90.0)
- removed the G1 at (332.5, 90.0)
- removed the G1 at (336.5, 90.0)
- removed the G1 at (340.5, 90.0)
- removed the G1 at (348.5, 90.0)
- removed the G1 at (308.5, 90.0)
- removed the G1 at (344.5, 90.0)
- removed the G1 at (300.5, 90.0)
- removed the G1 at (296.5, 90.0)
- removed the G1 at (292.5, 90.0)
- removed the G1 at (312.5, 90.0)
- removed the G1 at (316.5, 90.0)
- removed the G1 at (320.5, 90.0)
- removed the G1 at (328.5, 90.0)
- removed the G2 at (304.5, 123.0)
- removed the G2 at (324.5, 123.0)
- removed the G2 at (364.5, 123.0)
- removed the G2 at (368.5, 123.0)
- removed the G2 at (360.5, 123.0)
- removed the G2 at (356.5, 123.0)
- removed the G2 at (352.5, 123.0)
- removed the G2 at (332.5, 123.0)
- removed the G2 at (336.5, 123.0)
- removed the G2 at (340.5, 123.0)
- removed the G2 at (348.5, 123.0)
- removed the G2 at (308.5, 123.0)
- removed the G2 at (344.5, 123.0)
- removed the G2 at (300.5, 123.0)
- removed the G2 at (296.5, 123.0)
- removed the G2 at (292.5, 123.0)
- removed the G2 at (312.5, 123.0)
- removed the G2 at (316.5, 123.0)
- removed the G2 at (320.5, 123.0)
- removed the G2 at (328.5, 123.0)
- added D10: LED, my_parts:MADW__CHIPLED-0805, B.Cu at (300.5, 93.0)
- added D10: LED, my_parts:MADW__CHIPLED-0805, B.Cu at (320.5, 93.0)
- added D10: LED, my_parts:MADW__CHIPLED-0805, B.Cu at (360.5, 93.0)
- added D10: LED, my_parts:MADW__CHIPLED-0805, B.Cu at (364.5, 93.0)
- added D10: LED, my_parts:MADW__CHIPLED-0805, B.Cu at (356.5, 93.0)
- added D10: LED, my_parts:MADW__CHIPLED-0805, B.Cu at (352.5, 93.0)
- added D10: LED, my_parts:MADW__CHIPLED-0805, B.Cu at (368.5, 93.0)
- added D10: LED, my_parts:MADW__CHIPLED-0805, B.Cu at (348.5, 93.0)
- added D10: LED, my_parts:MADW__CHIPLED-0805, B.Cu at (332.5, 93.0)
- added D10: LED, my_parts:MADW__CHIPLED-0805, B.Cu at (336.5, 93.0)
- added D10: LED, my_parts:MADW__CHIPLED-0805, B.Cu at (344.5, 93.0)
- added D10: LED, my_parts:MADW__CHIPLED-0805, B.Cu at (304.5, 93.0)
- added D10: LED, my_parts:MADW__CHIPLED-0805, B.Cu at (340.5, 93.0)
- added D10: LED, my_parts:MADW__CHIPLED-0805, B.Cu at (296.5, 93.0)
- added D10: LED, my_parts:MADW__CHIPLED-0805, B.Cu at (292.5, 93.0)
- added D10: LED, my_parts:MADW__CHIPLED-0805, B.Cu at (308.5, 93.0)
- added D10: LED, my_parts:MADW__CHIPLED-0805, B.Cu at (328.5, 93.0)
- added D10: LED, my_parts:MADW__CHIPLED-0805, B.Cu at (312.5, 93.0)
- added D10: LED, my_parts:MADW__CHIPLED-0805, B.Cu at (316.5, 93.0)
- added D10: LED, my_parts:MADW__CHIPLED-0805, B.Cu at (324.5, 93.0)
- added D11: LED, my_parts:MADW__CHIPLED-0805, B.Cu at (300.5, 103.0)
- added D11: LED, my_parts:MADW__CHIPLED-0805, B.Cu at (320.5, 103.0)
- added D11: LED, my_parts:MADW__CHIPLED-0805, B.Cu at (360.5, 103.0)
- added D11: LED, my_parts:MADW__CHIPLED-0805, B.Cu at (364.5, 103.0)
- added D11: LED, my_parts:MADW__CHIPLED-0805, B.Cu at (356.5, 103.0)
- added D11: LED, my_parts:MADW__CHIPLED-0805, B.Cu at (352.5, 103.0)
- added D11: LED, my_parts:MADW__CHIPLED-0805, B.Cu at (368.5, 103.0)
- added D11: LED, my_parts:MADW__CHIPLED-0805, B.Cu at (348.5, 103.0)
- added D11: LED, my_parts:MADW__CHIPLED-0805, B.Cu at (332.5, 103.0)
- added D11: LED, my_parts:MADW__CHIPLED-0805, B.Cu at (336.5, 103.0)
- added D11: LED, my_parts:MADW__CHIPLED-0805, B.Cu at (344.5, 103.0)
- added D11: LED, my_parts:MADW__CHIPLED-0805, B.Cu at (304.5, 103.0)
- added D11: LED, my_parts:MADW__CHIPLED-0805, B.Cu at (340.5, 103.0)
- added D11: LED, my_parts:MADW__CHIPLED-0805, B.Cu at (296.5, 103.0)
- added D11: LED, my_parts:MADW__CHIPLED-0805, B.Cu at (292.5, 103.0)
- added D11: LED, my_parts:MADW__CHIPLED-0805, B.Cu at (308.5, 103.0)
- added D11: LED, my_parts:MADW__CHIPLED-0805, B.Cu at (328.5, 103.0)
- added D11: LED, my_parts:MADW__CHIPLED-0805, B.Cu at (312.5, 103.0)
- added D11: LED, my_parts:MADW__CHIPLED-0805, B.Cu at (316.5, 103.0)
- added D11: LED, my_parts:MADW__CHIPLED-0805, B.Cu at (324.5, 103.0)
- added D12: LED, my_parts:MADW__CHIPLED-0805, B.Cu at (300.5, 113.0)
- added D12: LED, my_parts:MADW__CHIPLED-0805, B.Cu at (320.5, 113.0)
- added D12: LED, my_parts:MADW__CHIPLED-0805, B.Cu at (360.5, 113.0)
- added D12: LED, my_parts:MADW__CHIPLED-0805, B.Cu at (364.5, 113.0)
- added D12: LED, my_parts:MADW__CHIPLED-0805, B.Cu at (356.5, 113.0)
- added D12: LED, my_parts:MADW__CHIPLED-0805, B.Cu at (352.5, 113.0)
- added D12: LED, my_parts:MADW__CHIPLED-0805, B.Cu at (368.5, 113.0)
- added D12: LED, my_parts:MADW__CHIPLED-0805, B.Cu at (348.5, 113.0)
- added D12: LED, my_parts:MADW__CHIPLED-0805, B.Cu at (332.5, 113.0)
- added D12: LED, my_parts:MADW__CHIPLED-0805, B.Cu at (336.5, 113.0)
- added D12: LED, my_parts:MADW__CHIPLED-0805, B.Cu at (344.5, 113.0)
- added D12: LED, my_parts:MADW__CHIPLED-0805, B.Cu at (304.5, 113.0)
- added D12: LED, my_parts:MADW__CHIPLED-0805, B.Cu at (340.5, 113.0)
- added D12: LED, my_parts:MADW__CHIPLED-0805, B.Cu at (296.5, 113.0)
- added D12: LED, my_parts:MADW__CHIPLED-0805, B.Cu at (292.5, 113.0)
- added D12: LED, my_parts:MADW__CHIPLED-0805, B.Cu at (308.5, 113.0)
- added D12: LED, my_parts:MADW__CHIPLED-0805, B.Cu at (328.5, 113.0)
- added D12: LED, my_parts:MADW__CHIPLED-0805, B.Cu at (312.5, 113.0)
- added D12: LED, my_parts:MADW__CHIPLED-0805, B.Cu at (316.5, 113.0)
- added D12: LED, my_parts:MADW__CHIPLED-0805, B.Cu at (324.5, 113.0)
- added D13: LED, my_parts:MADW__CHIPLED-0805, B.Cu at (300.5, 123.0)
- added D13: LED, my_parts:MADW__CHIPLED-0805, B.Cu at (320.5, 123.0)
- added D13: LED, my_parts:MADW__CHIPLED-0805, B.Cu at (360.5, 123.0)
- added D13: LED, my_parts:MADW__CHIPLED-0805, B.Cu at (364.5, 123.0)
- added D13: LED, my_parts:MADW__CHIPLED-0805, B.Cu at (356.5, 123.0)
- added D13: LED, my_parts:MADW__CHIPLED-0805, B.Cu at (352.5, 123.0)
- added D13: LED, my_parts:MADW__CHIPLED-0805, B.Cu at (368.5, 123.0)
- added D13: LED, my_parts:MADW__CHIPLED-0805, B.Cu at (348.5, 123.0)
- added D13: LED, my_parts:MADW__CHIPLED-0805, B.Cu at (332.5, 123.0)
- added D13: LED, my_parts:MADW__CHIPLED-0805, B.Cu at (336.5, 123.0)
- added D13: LED, my_parts:MADW__CHIPLED-0805, B.Cu at (344.5, 123.0)
- added D13: LED, my_parts:MADW__CHIPLED-0805, B.Cu at (304.5, 123.0)
- added D13: LED, my_parts:MADW__CHIPLED-0805, B.Cu at (340.5, 123.0)
- added D13: LED, my_parts:MADW__CHIPLED-0805, B.Cu at (296.5, 123.0)
- added D13: LED, my_parts:MADW__CHIPLED-0805, B.Cu at (292.5, 123.0)
- added D13: LED, my_parts:MADW__CHIPLED-0805, B.Cu at (308.5, 123.0)
- added D13: LED, my_parts:MADW__CHIPLED-0805, B.Cu at (328.5, 123.0)
- added D13: LED, my_parts:MADW__CHIPLED-0805, B.Cu at (312.5, 123.0)
- added D13: LED, my_parts:MADW__CHIPLED-0805, B.Cu at (316.5, 123.0)
- added D13: LED, my_parts:MADW__CHIPLED-0805, B.Cu at (324.5, 123.0)
- added D14: LED, my_parts:MADW__CHIPLED-0805, B.Cu at (300.5, 133.0)
- added D14: LED, my_parts:MADW__CHIPLED-0805, B.Cu at (320.5, 133.0)
- added D14: LED, my_parts:MADW__CHIPLED-0805, B.Cu at (360.5, 133.0)
- added D14: LED, my_parts:MADW__CHIPLED-0805, B.Cu at (364.5, 133.0)
- added D14: LED, my_parts:MADW__CHIPLED-0805, B.Cu at (356.5, 133.0)
- added D14: LED, my_parts:MADW__CHIPLED-0805, B.Cu at (352.5, 133.0)
- added D14: LED, my_parts:MADW__CHIPLED-0805, B.Cu at (368.5, 133.0)
- added D14: LED, my_parts:MADW__CHIPLED-0805, B.Cu at (348.5, 133.0)
- added D14: LED, my_parts:MADW__CHIPLED-0805, B.Cu at (332.5, 133.0)
- added D14: LED, my_parts:MADW__CHIPLED-0805, B.Cu at (336.5, 133.0)
- added D14: LED, my_parts:MADW__CHIPLED-0805, B.Cu at (344.5, 133.0)
- added D14: LED, my_parts:MADW__CHIPLED-0805, B.Cu at (304.5, 133.0)
- added D14: LED, my_parts:MADW__CHIPLED-0805, B.Cu at (340.5, 133.0)
- added D14: LED, my_parts:MADW__CHIPLED-0805, B.Cu at (296.5, 133.0)
- added D14: LED, my_parts:MADW__CHIPLED-0805, B.Cu at (292.5, 133.0)
- added D14: LED, my_parts:MADW__CHIPLED-0805, B.Cu at (308.5, 133.0)
- added D14: LED, my_parts:MADW__CHIPLED-0805, B.Cu at (328.5, 133.0)
- added D14: LED, my_parts:MADW__CHIPLED-0805, B.Cu at (312.5, 133.0)
- added D14: LED, my_parts:MADW__CHIPLED-0805, B.Cu at (316.5, 133.0)
- added D14: LED, my_parts:MADW__CHIPLED-0805, B.Cu at (324.5, 133.0)
- added D15: LED, my_parts:MADW__CHIPLED-0805, B.Cu at (300.5, 143.0)
- added D15: LED, my_parts:MADW__CHIPLED-0805, B.Cu at (320.5, 143.0)
- added D15: LED, my_parts:MADW__CHIPLED-0805, B.Cu at (360.5, 143.0)
- added D15: LED, my_parts:MADW__CHIPLED-0805, B.Cu at (364.5, 143.0)
- added D15: LED, my_parts:MADW__CHIPLED-0805, B.Cu at (356.5, 143.0)
- added D15: LED, my_parts:MADW__CHIPLED-0805, B.Cu at (352.5, 143.0)
- added D15: LED, my_parts:MADW__CHIPLED-0805, B.Cu at (368.5, 143.0)
- added D15: LED, my_parts:MADW__CHIPLED-0805, B.Cu at (348.5, 143.0)
- added D15: LED, my_parts:MADW__CHIPLED-0805, B.Cu at (332.5, 143.0)
- added D15: LED, my_parts:MADW__CHIPLED-0805, B.Cu at (336.5, 143.0)
- added D15: LED, my_parts:MADW__CHIPLED-0805, B.Cu at (344.5, 143.0)
- added D15: LED, my_parts:MADW__CHIPLED-0805, B.Cu at (304.5, 143.0)
- added D15: LED, my_parts:MADW__CHIPLED-0805, B.Cu at (340.5, 143.0)
- added D15: LED, my_parts:MADW__CHIPLED-0805, B.Cu at (296.5, 143.0)
- added D15: LED, my_parts:MADW__CHIPLED-0805, B.Cu at (292.5, 143.0)
- added D15: LED, my_parts:MADW__CHIPLED-0805, B.Cu at (308.5, 143.0)
- added D15: LED, my_parts:MADW__CHIPLED-0805, B.Cu at (328.5, 143.0)
- added D15: LED, my_parts:MADW__CHIPLED-0805, B.Cu at (312.5, 143.0)
- added D15: LED, my_parts:MADW__CHIPLED-0805, B.Cu at (316.5, 143.0)
- added D15: LED, my_parts:MADW__CHIPLED-0805, B.Cu at (324.5, 143.0)
- added D16: LED, my_parts:MADW__CHIPLED-0805, B.Cu at (300.5, 153.0)
- added D16: LED, my_parts:MADW__CHIPLED-0805, B.Cu at (320.5, 153.0)
- added D16: LED, my_parts:MADW__CHIPLED-0805, B.Cu at (360.5, 153.0)
- added D16: LED, my_parts:MADW__CHIPLED-0805, B.Cu at (364.5, 153.0)
- added D16: LED, my_parts:MADW__CHIPLED-0805, B.Cu at (356.5, 153.0)
- added D16: LED, my_parts:MADW__CHIPLED-0805, B.Cu at (352.5, 153.0)
- added D16: LED, my_parts:MADW__CHIPLED-0805, B.Cu at (368.5, 153.0)
- added D16: LED, my_parts:MADW__CHIPLED-0805, B.Cu at (348.5, 153.0)
- added D16: LED, my_parts:MADW__CHIPLED-0805, B.Cu at (332.5, 153.0)
- added D16: LED, my_parts:MADW__CHIPLED-0805, B.Cu at (336.5, 153.0)
- added D16: LED, my_parts:MADW__CHIPLED-0805, B.Cu at (344.5, 153.0)
- added D16: LED, my_parts:MADW__CHIPLED-0805, B.Cu at (304.5, 153.0)
- added D16: LED, my_parts:MADW__CHIPLED-0805, B.Cu at (340.5, 153.0)
- added D16: LED, my_parts:MADW__CHIPLED-0805, B.Cu at (296.5, 153.0)
- added D16: LED, my_parts:MADW__CHIPLED-0805, B.Cu at (292.5, 153.0)
- added D16: LED, my_parts:MADW__CHIPLED-0805, B.Cu at (308.5, 153.0)
- added D16: LED, my_parts:MADW__CHIPLED-0805, B.Cu at (328.5, 153.0)
- added D16: LED, my_parts:MADW__CHIPLED-0805, B.Cu at (312.5, 153.0)
- added D16: LED, my_parts:MADW__CHIPLED-0805, B.Cu at (316.5, 153.0)
- added D16: LED, my_parts:MADW__CHIPLED-0805, B.Cu at (324.5, 153.0)
- added D17: LED, my_parts:MADW__CHIPLED-0805, B.Cu at (300.5, 163.0)
- added D17: LED, my_parts:MADW__CHIPLED-0805, B.Cu at (320.5, 163.0)
- added D17: LED, my_parts:MADW__CHIPLED-0805, B.Cu at (360.5, 163.0)
- added D17: LED, my_parts:MADW__CHIPLED-0805, B.Cu at (364.5, 163.0)
- added D17: LED, my_parts:MADW__CHIPLED-0805, B.Cu at (356.5, 163.0)
- added D17: LED, my_parts:MADW__CHIPLED-0805, B.Cu at (352.5, 163.0)
- added D17: LED, my_parts:MADW__CHIPLED-0805, B.Cu at (368.5, 163.0)
- added D17: LED, my_parts:MADW__CHIPLED-0805, B.Cu at (348.5, 163.0)
- added D17: LED, my_parts:MADW__CHIPLED-0805, B.Cu at (332.5, 163.0)
- added D17: LED, my_parts:MADW__CHIPLED-0805, B.Cu at (336.5, 163.0)
- added D17: LED, my_parts:MADW__CHIPLED-0805, B.Cu at (344.5, 163.0)
- added D17: LED, my_parts:MADW__CHIPLED-0805, B.Cu at (304.5, 163.0)
- added D17: LED, my_parts:MADW__CHIPLED-0805, B.Cu at (340.5, 163.0)
- added D17: LED, my_parts:MADW__CHIPLED-0805, B.Cu at (296.5, 163.0)
- added D17: LED, my_parts:MADW__CHIPLED-0805, B.Cu at (292.5, 163.0)
- added D17: LED, my_parts:MADW__CHIPLED-0805, B.Cu at (308.5, 163.0)
- added D17: LED, my_parts:MADW__CHIPLED-0805, B.Cu at (328.5, 163.0)
- added D17: LED, my_parts:MADW__CHIPLED-0805, B.Cu at (312.5, 163.0)
- added D17: LED, my_parts:MADW__CHIPLED-0805, B.Cu at (316.5, 163.0)
- added D17: LED, my_parts:MADW__CHIPLED-0805, B.Cu at (324.5, 163.0)
- added D18: LED, my_parts:MADW__CHIPLED-0805, B.Cu at (300.5, 173.0)
- added D18: LED, my_parts:MADW__CHIPLED-0805, B.Cu at (320.5, 173.0)
- added D18: LED, my_parts:MADW__CHIPLED-0805, B.Cu at (360.5, 173.0)
- added D18: LED, my_parts:MADW__CHIPLED-0805, B.Cu at (364.5, 173.0)
- added D18: LED, my_parts:MADW__CHIPLED-0805, B.Cu at (356.5, 173.0)
- added D18: LED, my_parts:MADW__CHIPLED-0805, B.Cu at (352.5, 173.0)
- added D18: LED, my_parts:MADW__CHIPLED-0805, B.Cu at (368.5, 173.0)
- added D18: LED, my_parts:MADW__CHIPLED-0805, B.Cu at (348.5, 173.0)
- added D18: LED, my_parts:MADW__CHIPLED-0805, B.Cu at (332.5, 173.0)
- added D18: LED, my_parts:MADW__CHIPLED-0805, B.Cu at (336.5, 173.0)
- added D18: LED, my_parts:MADW__CHIPLED-0805, B.Cu at (344.5, 173.0)
- added D18: LED, my_parts:MADW__CHIPLED-0805, B.Cu at (304.5, 173.0)
- added D18: LED, my_parts:MADW__CHIPLED-0805, B.Cu at (340.5, 173.0)
- added D18: LED, my_parts:MADW__CHIPLED-0805, B.Cu at (296.5, 173.0)
- added D18: LED, my_parts:MADW__CHIPLED-0805, B.Cu at (292.5, 173.0)
- added D18: LED, my_parts:MADW__CHIPLED-0805, B.Cu at (308.5, 173.0)
- added D18: LED, my_parts:MADW__CHIPLED-0805, B.Cu at (328.5, 173.0)
- added D18: LED, my_parts:MADW__CHIPLED-0805, B.Cu at (312.5, 173.0)
- added D18: LED, my_parts:MADW__CHIPLED-0805, B.Cu at (316.5, 173.0)
- added D18: LED, my_parts:MADW__CHIPLED-0805, B.Cu at (324.5, 173.0)
- added G1: LED_smile_silkscreen_3mm, led-smile:LED_smile_silkscreen_3mm, B.Cu at (300.6, 98.1)
- added G1: LED_smile_silkscreen_3mm, led-smile:LED_smile_silkscreen_3mm, B.Cu at (320.6, 98.1)
- added G1: LED_smile_silkscreen_3mm, led-smile:LED_smile_silkscreen_3mm, B.Cu at (360.6, 98.1)
- added G1: LED_smile_silkscreen_3mm, led-smile:LED_smile_silkscreen_3mm, B.Cu at (364.6, 98.1)
- added G1: LED_smile_silkscreen_3mm, led-smile:LED_smile_silkscreen_3mm, B.Cu at (356.6, 98.1)
- added G1: LED_smile_silkscreen_3mm, led-smile:LED_smile_silkscreen_3mm, B.Cu at (352.6, 98.1)
- added G1: LED_smile_silkscreen_3mm, led-smile:LED_smile_silkscreen_3mm, B.Cu at (368.6, 98.1)
- added G1: LED_smile_silkscreen_3mm, led-smile:LED_smile_silkscreen_3mm, B.Cu at (348.6, 98.1)
- added G1: LED_smile_silkscreen_3mm, led-smile:LED_smile_silkscreen_3mm, B.Cu at (332.6, 98.1)
- added G1: LED_smile_silkscreen_3mm, led-smile:LED_smile_silkscreen_3mm, B.Cu at (336.6, 98.1)
- added G1: LED_smile_silkscreen_3mm, led-smile:LED_smile_silkscreen_3mm, B.Cu at (344.6, 98.1)
- added G1: LED_smile_silkscreen_3mm, led-smile:LED_smile_silkscreen_3mm, B.Cu at (304.6, 98.1)
- added G1: LED_smile_silkscreen_3mm, led-smile:LED_smile_silkscreen_3mm, B.Cu at (340.6, 98.1)
- added G1: LED_smile_silkscreen_3mm, led-smile:LED_smile_silkscreen_3mm, B.Cu at (296.6, 98.1)
- added G1: LED_smile_silkscreen_3mm, led-smile:LED_smile_silkscreen_3mm, B.Cu at (292.6, 98.1)
- added G1: LED_smile_silkscreen_3mm, led-smile:LED_smile_silkscreen_3mm, B.Cu at (308.6, 98.1)
- added G1: LED_smile_silkscreen_3mm, led-smile:LED_smile_silkscreen_3mm, B.Cu at (328.6, 98.1)
- added G1: LED_smile_silkscreen_3mm, led-smile:LED_smile_silkscreen_3mm, B.Cu at (312.6, 98.1)
- added G1: LED_smile_silkscreen_3mm, led-smile:LED_smile_silkscreen_3mm, B.Cu at (316.6, 98.1)
- added G1: LED_smile_silkscreen_3mm, led-smile:LED_smile_silkscreen_3mm, B.Cu at (324.6, 98.1)
- added G2: OSHW-logo_silkscreen_3mm, oshw-logo:OSHW-logo_silkscreen_3mm, B.Cu at (300.5, 128.1)
- added G2: OSHW-logo_silkscreen_3mm, oshw-logo:OSHW-logo_silkscreen_3mm, B.Cu at (320.5, 128.1)
- added G2: OSHW-logo_silkscreen_3mm, oshw-logo:OSHW-logo_silkscreen_3mm, B.Cu at (360.5, 128.1)
- added G2: OSHW-logo_silkscreen_3mm, oshw-logo:OSHW-logo_silkscreen_3mm, B.Cu at (364.5, 128.1)
- added G2: OSHW-logo_silkscreen_3mm, oshw-logo:OSHW-logo_silkscreen_3mm, B.Cu at (356.5, 128.1)
- added G2: OSHW-logo_silkscreen_3mm, oshw-logo:OSHW-logo_silkscreen_3mm, B.Cu at (352.5, 128.1)
- added G2: OSHW-logo_silkscreen_3mm, oshw-logo:OSHW-logo_silkscreen_3mm, B.Cu at (368.5, 128.1)
- added G2: OSHW-logo_silkscreen_3mm, oshw-logo:OSHW-logo_silkscreen_3mm, B.Cu at (348.5, 128.1)
- added G2: OSHW-logo_silkscreen_3mm, oshw-logo:OSHW-logo_silkscreen_3mm, B.Cu at (332.5, 128.1)
- added G2: OSHW-logo_silkscreen_3mm, oshw-logo:OSHW-logo_silkscreen_3mm, B.Cu at (336.5, 128.1)
- added G2: OSHW-logo_silkscreen_3mm, oshw-logo:OSHW-logo_silkscreen_3mm, B.Cu at (344.5, 128.1)
- added G2: OSHW-logo_silkscreen_3mm, oshw-logo:OSHW-logo_silkscreen_3mm, B.Cu at (304.5, 128.1)
- added G2: OSHW-logo_silkscreen_3mm, oshw-logo:OSHW-logo_silkscreen_3mm, B.Cu at (340.5, 128.1)
- added G2: OSHW-logo_silkscreen_3mm, oshw-logo:OSHW-logo_silkscreen_3mm, B.Cu at (296.5, 128.1)
- added G2: OSHW-logo_silkscreen_3mm, oshw-logo:OSHW-logo_silkscreen_3mm, B.Cu at (292.5, 128.1)
- added G2: OSHW-logo_silkscreen_3mm, oshw-logo:OSHW-logo_silkscreen_3mm, B.Cu at (308.5, 128.1)
- added G2: OSHW-logo_silkscreen_3mm, oshw-logo:OSHW-logo_silkscreen_3mm, B.Cu at (328.5, 128.1)
- added G2: OSHW-logo_silkscreen_3mm, oshw-logo:OSHW-logo_silkscreen_3mm, B.Cu at (312.5, 128.1)
- added G2: OSHW-logo_silkscreen_3mm, oshw-logo:OSHW-logo_silkscreen_3mm, B.Cu at (316.5, 128.1)
- added G2: OSHW-logo_silkscreen_3mm, oshw-logo:OSHW-logo_silkscreen_3mm, B.Cu at (324.5, 128.1)
- added P10: CONN_2, my_parts:MADW__SIL-2, B.Cu at (300.5, 146.5)
- added P10: CONN_2, my_parts:MADW__SIL-2, B.Cu at (320.5, 146.5)
- added P10: CONN_2, my_parts:MADW__SIL-2, B.Cu at (360.5, 146.5)
- added P10: CONN_2, my_parts:MADW__SIL-2, B.Cu at (364.5, 146.5)
- added P10: CONN_2, my_parts:MADW__SIL-2, B.Cu at (356.5, 146.5)
- added P10: CONN_2, my_parts:MADW__SIL-2, B.Cu at (352.5, 146.5)
- added P10: CONN_2, my_parts:MADW__SIL-2, B.Cu at (368.5, 146.5)
- added P10: CONN_2, my_parts:MADW__SIL-2, B.Cu at (348.5, 146.5)
- added P10: CONN_2, my_parts:MADW__SIL-2, B.Cu at (332.5, 146.5)
- added P10: CONN_2, my_parts:MADW__SIL-2, B.Cu at (336.5, 146.5)
- added P10: CONN_2, my_parts:MADW__SIL-2, B.Cu at (344.5, 146.5)
- added P10: CONN_2, my_parts:MADW__SIL-2, B.Cu at (304.5, 146.5)
- added P10: CONN_2, my_parts:MADW__SIL-2, B.Cu at (340.5, 146.5)
- added P10: CONN_2, my_parts:MADW__SIL-2, B.Cu at (296.5, 146.5)
- added P10: CONN_2, my_parts:MADW__SIL-2, B.Cu at (292.5, 146.5)
- added P10: CONN_2, my_parts:MADW__SIL-2, B.Cu at (308.5, 146.5)
- added P10: CONN_2, my_parts:MADW__SIL-2, B.Cu at (328.5, 146.5)
- added P10: CONN_2, my_parts:MADW__SIL-2, B.Cu at (312.5, 146.5)
- added P10: CONN_2, my_parts:MADW__SIL-2, B.Cu at (316.5, 146.5)
- added P10: CONN_2, my_parts:MADW__SIL-2, B.Cu at (324.5, 146.5)
- added P11: CONN_2, my_parts:MADW__SIL-2, B.Cu at (300.5, 149.5)
- added P11: CONN_2, my_parts:MADW__SIL-2, B.Cu at (320.5, 149.5)
- added P11: CONN_2, my_parts:MADW__SIL-2, B.Cu at (360.5, 149.5)
- added P11: CONN_2, my_parts:MADW__SIL-2, B.Cu at (364.5, 149.5)
- added P11: CONN_2, my_parts:MADW__SIL-2, B.Cu at (356.5, 149.5)
- added P11: CONN_2, my_parts:MADW__SIL-2, B.Cu at (352.5, 149.5)
- added P11: CONN_2, my_parts:MADW__SIL-2, B.Cu at (368.5, 149.5)
- added P11: CONN_2, my_parts:MADW__SIL-2, B.Cu at (348.5, 149.5)
- added P11: CONN_2, my_parts:MADW__SIL-2, B.Cu at (332.5, 149.5)
- added P11: CONN_2, my_parts:MADW__SIL-2, B.Cu at (336.5, 149.5)
- added P11: CONN_2, my_parts:MADW__SIL-2, B.Cu at (344.5, 149.5)
- added P11: CONN_2, my_parts:MADW__SIL-2, B.Cu at (304.5, 149.5)
- added P11: CONN_2, my_parts:MADW__SIL-2, B.Cu at (340.5, 149.5)
- added P11: CONN_2, my_parts:MADW__SIL-2, B.Cu at (296.5, 149.5)
- added P11: CONN_2, my_parts:MADW__SIL-2, B.Cu at (292.5, 149.5)
- added P11: CONN_2, my_parts:MADW__SIL-2, B.Cu at (308.5, 149.5)
- added P11: CONN_2, my_parts:MADW__SIL-2, B.Cu at (328.5, 149.5)
- added P11: CONN_2, my_parts:MADW__SIL-2, B.Cu at (312.5, 149.5)
- added P11: CONN_2, my_parts:MADW__SIL-2, B.Cu at (316.5, 149.5)
- added P11: CONN_2, my_parts:MADW__SIL-2, B.Cu at (324.5, 149.5)
- added P12: CONN_2, my_parts:MADW__SIL-2, B.Cu at (300.5, 176.5)
- added P12: CONN_2, my_parts:MADW__SIL-2, B.Cu at (320.5, 176.5)
- added P12: CONN_2, my_parts:MADW__SIL-2, B.Cu at (360.5, 176.5)
- added P12: CONN_2, my_parts:MADW__SIL-2, B.Cu at (364.5, 176.5)
- added P12: CONN_2, my_parts:MADW__SIL-2, B.Cu at (356.5, 176.5)
- added P12: CONN_2, my_parts:MADW__SIL-2, B.Cu at (352.5, 176.5)
- added P12: CONN_2, my_parts:MADW__SIL-2, B.Cu at (368.5, 176.5)
- added P12: CONN_2, my_parts:MADW__SIL-2, B.Cu at (348.5, 176.5)
- added P12: CONN_2, my_parts:MADW__SIL-2, B.Cu at (332.5, 176.5)
- added P12: CONN_2, my_parts:MADW__SIL-2, B.Cu at (336.5, 176.5)
- added P12: CONN_2, my_parts:MADW__SIL-2, B.Cu at (344.5, 176.5)
- added P12: CONN_2, my_parts:MADW__SIL-2, B.Cu at (304.5, 176.5)
- added P12: CONN_2, my_parts:MADW__SIL-2, B.Cu at (340.5, 176.5)
- added P12: CONN_2, my_parts:MADW__SIL-2, B.Cu at (296.5, 176.5)
- added P12: CONN_2, my_parts:MADW__SIL-2, B.Cu at (292.5, 176.5)
- added P12: CONN_2, my_parts:MADW__SIL-2, B.Cu at (308.5, 176.5)
- added P12: CONN_2, my_parts:MADW__SIL-2, B.Cu at (328.5, 176.5)
- added P12: CONN_2, my_parts:MADW__SIL-2, B.Cu at (312.5, 176.5)
- added P12: CONN_2, my_parts:MADW__SIL-2, B.Cu at (316.5, 176.5)
- added P12: CONN_2, my_parts:MADW__SIL-2, B.Cu at (324.5, 176.5)
- added P7: CONN_2, my_parts:MADW__SIL-2, B.Cu at (300.5, 89.5)
- added P7: CONN_2, my_parts:MADW__SIL-2, B.Cu at (320.5, 89.5)
- added P7: CONN_2, my_parts:MADW__SIL-2, B.Cu at (360.5, 89.5)
- added P7: CONN_2, my_parts:MADW__SIL-2, B.Cu at (364.5, 89.5)
- added P7: CONN_2, my_parts:MADW__SIL-2, B.Cu at (356.5, 89.5)
- added P7: CONN_2, my_parts:MADW__SIL-2, B.Cu at (352.5, 89.5)
- added P7: CONN_2, my_parts:MADW__SIL-2, B.Cu at (368.5, 89.5)
- added P7: CONN_2, my_parts:MADW__SIL-2, B.Cu at (348.5, 89.5)
- added P7: CONN_2, my_parts:MADW__SIL-2, B.Cu at (332.5, 89.5)
- added P7: CONN_2, my_parts:MADW__SIL-2, B.Cu at (336.5, 89.5)
- added P7: CONN_2, my_parts:MADW__SIL-2, B.Cu at (344.5, 89.5)
- added P7: CONN_2, my_parts:MADW__SIL-2, B.Cu at (304.5, 89.5)
- added P7: CONN_2, my_parts:MADW__SIL-2, B.Cu at (340.5, 89.5)
- added P7: CONN_2, my_parts:MADW__SIL-2, B.Cu at (296.5, 89.5)
- added P7: CONN_2, my_parts:MADW__SIL-2, B.Cu at (292.5, 89.5)
- added P7: CONN_2, my_parts:MADW__SIL-2, B.Cu at (308.5, 89.5)
- added P7: CONN_2, my_parts:MADW__SIL-2, B.Cu at (328.5, 89.5)
- added P7: CONN_2, my_parts:MADW__SIL-2, B.Cu at (312.5, 89.5)
- added P7: CONN_2, my_parts:MADW__SIL-2, B.Cu at (316.5, 89.5)
- added P7: CONN_2, my_parts:MADW__SIL-2, B.Cu at (324.5, 89.5)
- added P8: CONN_2, my_parts:MADW__SIL-2, B.Cu at (300.5, 116.5)
- added P8: CONN_2, my_parts:MADW__SIL-2, B.Cu at (320.5, 116.5)
- added P8: CONN_2, my_parts:MADW__SIL-2, B.Cu at (360.5, 116.5)
- added P8: CONN_2, my_parts:MADW__SIL-2, B.Cu at (364.5, 116.5)
- added P8: CONN_2, my_parts:MADW__SIL-2, B.Cu at (356.5, 116.5)
- added P8: CONN_2, my_parts:MADW__SIL-2, B.Cu at (352.5, 116.5)
- added P8: CONN_2, my_parts:MADW__SIL-2, B.Cu at (368.5, 116.5)
- added P8: CONN_2, my_parts:MADW__SIL-2, B.Cu at (348.5, 116.5)
- added P8: CONN_2, my_parts:MADW__SIL-2, B.Cu at (332.5, 116.5)
- added P8: CONN_2, my_parts:MADW__SIL-2, B.Cu at (336.5, 116.5)
- added P8: CONN_2, my_parts:MADW__SIL-2, B.Cu at (344.5, 116.5)
- added P8: CONN_2, my_parts:MADW__SIL-2, B.Cu at (304.5, 116.5)
- added P8: CONN_2, my_parts:MADW__SIL-2, B.Cu at (340.5, 116.5)
- added P8: CONN_2, my_parts:MADW__SIL-2, B.Cu at (296.5, 116.5)
- added P8: CONN_2, my_parts:MADW__SIL-2, B.Cu at (292.5, 116.5)
- added P8: CONN_2, my_parts:MADW__SIL-2, B.Cu at (308.5, 116.5)
- added P8: CONN_2, my_parts:MADW__SIL-2, B.Cu at (328.5, 116.5)
- added P8: CONN_2, my_parts:MADW__SIL-2, B.Cu at (312.5, 116.5)
- added P8: CONN_2, my_parts:MADW__SIL-2, B.Cu at (316.5, 116.5)
- added P8: CONN_2, my_parts:MADW__SIL-2, B.Cu at (324.5, 116.5)
- added P9: CONN_2, my_parts:MADW__SIL-2, B.Cu at (300.5, 119.5)
- added P9: CONN_2, my_parts:MADW__SIL-2, B.Cu at (320.5, 119.5)
- added P9: CONN_2, my_parts:MADW__SIL-2, B.Cu at (360.5, 119.5)
- added P9: CONN_2, my_parts:MADW__SIL-2, B.Cu at (364.5, 119.5)
- added P9: CONN_2, my_parts:MADW__SIL-2, B.Cu at (356.5, 119.5)
- added P9: CONN_2, my_parts:MADW__SIL-2, B.Cu at (352.5, 119.5)
- added P9: CONN_2, my_parts:MADW__SIL-2, B.Cu at (368.5, 119.5)
- added P9: CONN_2, my_parts:MADW__SIL-2, B.Cu at (348.5, 119.5)
- added P9: CONN_2, my_parts:MADW__SIL-2, B.Cu at (332.5, 119.5)
- added P9: CONN_2, my_parts:MADW__SIL-2, B.Cu at (336.5, 119.5)
- added P9: CONN_2, my_parts:MADW__SIL-2, B.Cu at (344.5, 119.5)
- added P9: CONN_2, my_parts:MADW__SIL-2, B.Cu at (304.5, 119.5)
- added P9: CONN_2, my_parts:MADW__SIL-2, B.Cu at (340.5, 119.5)
- added P9: CONN_2, my_parts:MADW__SIL-2, B.Cu at (296.5, 119.5)
- added P9: CONN_2, my_parts:MADW__SIL-2, B.Cu at (292.5, 119.5)
- added P9: CONN_2, my_parts:MADW__SIL-2, B.Cu at (308.5, 119.5)
- added P9: CONN_2, my_parts:MADW__SIL-2, B.Cu at (328.5, 119.5)
- added P9: CONN_2, my_parts:MADW__SIL-2, B.Cu at (312.5, 119.5)
- added P9: CONN_2, my_parts:MADW__SIL-2, B.Cu at (316.5, 119.5)
- added P9: CONN_2, my_parts:MADW__SIL-2, B.Cu at (324.5, 119.5)
- added R4: R, my_parts:MADW__R0603_2, B.Cu at (300.5, 107.9)
- added R4: R, my_parts:MADW__R0603_2, B.Cu at (320.5, 107.9)
- added R4: R, my_parts:MADW__R0603_2, B.Cu at (360.5, 107.9)
- added R4: R, my_parts:MADW__R0603_2, B.Cu at (364.5, 107.9)
- added R4: R, my_parts:MADW__R0603_2, B.Cu at (356.5, 107.9)
- added R4: R, my_parts:MADW__R0603_2, B.Cu at (352.5, 107.9)
- added R4: R, my_parts:MADW__R0603_2, B.Cu at (368.5, 107.9)
- added R4: R, my_parts:MADW__R0603_2, B.Cu at (348.5, 107.9)
- added R4: R, my_parts:MADW__R0603_2, B.Cu at (332.5, 107.9)
- added R4: R, my_parts:MADW__R0603_2, B.Cu at (336.5, 107.9)
- added R4: R, my_parts:MADW__R0603_2, B.Cu at (344.5, 107.9)
- added R4: R, my_parts:MADW__R0603_2, B.Cu at (304.5, 107.9)
- added R4: R, my_parts:MADW__R0603_2, B.Cu at (340.5, 107.9)
- added R4: R, my_parts:MADW__R0603_2, B.Cu at (296.5, 107.9)
- added R4: R, my_parts:MADW__R0603_2, B.Cu at (292.5, 107.9)
- added R4: R, my_parts:MADW__R0603_2, B.Cu at (308.5, 107.9)
- added R4: R, my_parts:MADW__R0603_2, B.Cu at (328.5, 107.9)
- added R4: R, my_parts:MADW__R0603_2, B.Cu at (312.5, 107.9)
- added R4: R, my_parts:MADW__R0603_2, B.Cu at (316.5, 107.9)
- added R4: R, my_parts:MADW__R0603_2, B.Cu at (324.5, 107.9)
- added R5: R, my_parts:MADW__R0603_2, B.Cu at (300.5, 137.9)
- added R5: R, my_parts:MADW__R0603_2, B.Cu at (320.5, 137.9)
- added R5: R, my_parts:MADW__R0603_2, B.Cu at (360.5, 137.9)
- added R5: R, my_parts:MADW__R0603_2, B.Cu at (364.5, 137.9)
- added R5: R, my_parts:MADW__R0603_2, B.Cu at (356.5, 137.9)
- added R5: R, my_parts:MADW__R0603_2, B.Cu at (352.5, 137.9)
- added R5: R, my_parts:MADW__R0603_2, B.Cu at (368.5, 137.9)
- added R5: R, my_parts:MADW__R0603_2, B.Cu at (348.5, 137.9)
- added R5: R, my_parts:MADW__R0603_2, B.Cu at (332.5, 137.9)
- added R5: R, my_parts:MADW__R0603_2, B.Cu at (336.5, 137.9)
- added R5: R, my_parts:MADW__R0603_2, B.Cu at (344.5, 137.9)
- added R5: R, my_parts:MADW__R0603_2, B.Cu at (304.5, 137.9)
- added R5: R, my_parts:MADW__R0603_2, B.Cu at (340.5, 137.9)
- added R5: R, my_parts:MADW__R0603_2, B.Cu at (296.5, 137.9)
- added R5: R, my_parts:MADW__R0603_2, B.Cu at (292.5, 137.9)
- added R5: R, my_parts:MADW__R0603_2, B.Cu at (308.5, 137.9)
- added R5: R, my_parts:MADW__R0603_2, B.Cu at (328.5, 137.9)
- added R5: R, my_parts:MADW__R0603_2, B.Cu at (312.5, 137.9)
- added R5: R, my_parts:MADW__R0603_2, B.Cu at (316.5, 137.9)
- added R5: R, my_parts:MADW__R0603_2, B.Cu at (324.5, 137.9)
- added R6: R, my_parts:MADW__R0603_2, B.Cu at (300.5, 167.9)
- added R6: R, my_parts:MADW__R0603_2, B.Cu at (320.5, 167.9)
- added R6: R, my_parts:MADW__R0603_2, B.Cu at (360.5, 167.9)
- added R6: R, my_parts:MADW__R0603_2, B.Cu at (364.5, 167.9)
- added R6: R, my_parts:MADW__R0603_2, B.Cu at (356.5, 167.9)
- added R6: R, my_parts:MADW__R0603_2, B.Cu at (352.5, 167.9)
- added R6: R, my_parts:MADW__R0603_2, B.Cu at (368.5, 167.9)
- added R6: R, my_parts:MADW__R0603_2, B.Cu at (348.5, 167.9)
- added R6: R, my_parts:MADW__R0603_2, B.Cu at (332.5, 167.9)
- added R6: R, my_parts:MADW__R0603_2, B.Cu at (336.5, 167.9)
- added R6: R, my_parts:MADW__R0603_2, B.Cu at (344.5, 167.9)
- added R6: R, my_parts:MADW__R0603_2, B.Cu at (304.5, 167.9)
- added R6: R, my_parts:MADW__R0603_2, B.Cu at (340.5, 167.9)
- added R6: R, my_parts:MADW__R0603_2, B.Cu at (296.5, 167.9)
- added R6: R, my_parts:MADW__R0603_2, B.Cu at (292.5, 167.9)
- added R6: R, my_parts:MADW__R0603_2, B.Cu at (308.5, 167.9)
- added R6: R, my_parts:MADW__R0603_2, B.Cu at (328.5, 167.9)
- added R6: R, my_parts:MADW__R0603_2, B.Cu at (312.5, 167.9)
- added R6: R, my_parts:MADW__R0603_2, B.Cu at (316.5, 167.9)
- added R6: R, my_parts:MADW__R0603_2, B.Cu at (324.5, 167.9)
Routing:
- net /GND: track 1893.7 -> 3916.7 mm
- net /VCC: track 1920.9 -> 3876.0 mm
- net Net-(D10-Pad2): track 0.00 -> 158.0 mm
- net Net-(D13-Pad2): track 0.00 -> 158.0 mm
- net Net-(D16-Pad2): track 0.00 -> 158.0 mm
- net Net-(D18-Pad1): track 0.00 -> 64.1 mm
- net Net-(D15-Pad1): track 0.00 -> 64.1 mm
- net Net-(D12-Pad1): track 0.00 -> 64.1 mm
- net Net-(D11-Pad2): track 0.00 -> 60.1 mm
- net Net-(D17-Pad2): track 0.00 -> 60.1 mm
- net Net-(D14-Pad2): track 0.00 -> 60.1 mm
Other:
- net class Default: clearance 0.1524 -> 0.2032
- net class Power: clearance 0.1524 -> 0.2032
- rule trace_clearance: 0.1524 -> 0.2032
- rule via_min_drill: 0.3 -> 0.3302
- rule via_min_size: 0.6 -> 0.635
- board text added: "2014 V0.20.a"
- board text removed: "+ -"
- board text removed: "V0.10.b"
